File: tamagotchi.brd (EAGLE design)
At the start: 31.8 x 31.8 mm, 7 parts, among them U1 ATTINY84-20SSU

Commit message: gerber
Parts:
- removed OLED_CONN: 1x04 VERT FEMALE, PiB_connectors:HDRVR4W75P254_1X4_1066X254X850B
- moved S1 3.30 mm to (15.9, 23.7)
- moved BT1 1.00 mm to (15.9, 12.0)
- moved LS1 1.00 mm to (5.86, 21.5)
Connections:
- net 3V: no longer OLED_CONN.2
- net GND: no longer OLED_CONN.1
- net MISO: now also JP1.4; no longer JP1.1
- net PIEZO: now also U1.10; no longer U1.4
- net RST: now also U1.4; no longer U1.10
- net SCL/SCK: no longer OLED_CONN.3
- net SDA/MOSI: now also JP1.1; no longer JP1.4, OLED_CONN.4
Routing:
- net PIEZO: track 8.15 -> 23.4 mm
- net N$2: track 49.5 -> 34.5 mm
- net RST: track 9.40 -> 21.9 mm
- net MISO: track 20.9 -> 16.3 mm
- net SDA/MOSI: track 24.5 -> 25.9 mm, vias 0 -> 1
- net N$1: track 14.4 -> 15.2 mm
- net 3V: track 22.5 -> 22.0 mm, vias 0 -> 1
- net SCL/SCK: track 22.1 -> 22.4 mm, vias 0 -> 1
Other:
- board text added: "ATTINY84"
- board text added: "BATTERY CR2032"
- board text added: "BZR"
- board text added: "GND"
- board text added: "R1"
- board text added: "S1"
- board text added: "SCL"
- board text added: "SDA"
- board text added: "VCC"

Commit message: code, updated brd
Routing:
- net SCL/SCK: track 22.4 -> 35.7 mm
- net GND: track 0.00 -> 4.85 mm
Changed lines of the file:
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@@
 <drawing>
 <settings>
-<setting alwaysvectorfont="yes"/>
+<setting alwaysvectorfont="no"/>
 <setting verticaltext="up"/>
 </settings>
@@
 </polygon>
 <via x="12.065" y="27" extent="1-16" drill="1.7" diameter="2.3"/>
+<wire x1="22.825" y1="16.56" x2="26.225" y2="19.96" width="0.3048" layer="1"/>
+<wire x1="26.225" y1="19.96" x2="26.27" y2="19.96" width="0.3048" layer="1"/>
 </signal>
 <signal name="3V">
@@
 <wire x1="17.531675" y1="27" x2="19.511875" y2="25.0198" width="0.4064" layer="16"/>
 <wire x1="19.511875" y1="25.0198" x2="21.2102" y2="25.0198" width="0.4064" layer="16"/>
-<wire x1="23.8678375" y1="10.8498" x2="23.4648" y2="10.8498" width="0.4064" layer="1"/>
-<wire x1="23.4648" y1="10.8498" x2="22.825" y2="10.21" width="0.4064" layer="1"/>
-<wire x1="23.73" y1="22.5" x2="23.73" y2="21.72013125" width="0.4064" layer="1"/>
-<wire x1="23.73" y1="21.72013125" x2="24.9746" y2="20.47553125" width="0.4064" layer="1"/>
-<wire x1="24.9746" y1="20.47553125" x2="24.9746" y2="11.9565625" width="0.4064" layer="1"/>
-<wire x1="24.9746" y1="11.9565625" x2="23.8678375" y2="10.8498" width="0.4064" layer="1"/>
+<wire x1="25.77550625" y1="23.6938" x2="26.76449375" y2="23.6938" width="0.3048" layer="1"/>
+<wire x1="23.8468" y1="8.3606" x2="21.8606" y2="8.3606" width="0.3048" layer="1"/>
+<wire x1="21.8606" y1="8.3606" x2="21.5" y2="8" width="0.3048" layer="1"/>
+<wire x1="26.76449375" y1="23.6938" x2="27.9972" y2="22.46109375" width="0.3048" layer="1"/>
+<wire x1="27.9972" y1="22.46109375" x2="27.9972" y2="12.511" width="0.3048" layer="1"/>
+<wire x1="27.9972" y1="12.511" x2="23.8468" y2="8.3606" width="0.3048" layer="1"/>
+<wire x1="23.73" y1="22.5" x2="24.58170625" y2="22.5" width="0.3048" layer="1"/>
+<wire x1="24.58170625" y1="22.5" x2="25.77550625" y2="23.6938" width="0.3048" layer="1"/>
+<wire x1="21.5" y1="8" x2="21" y2="8" width="0.3048" layer="1"/>
+<wire x1="21.8032" y1="9.5194" x2="22.1344" y2="9.5194" width="0.3048" layer="1"/>
+<wire x1="22.1344" y1="9.5194" x2="22.825" y2="10.21" width="0.3048" layer="1"/>
+<wire x1="21" y1="8" x2="21" y2="8.7162" width="0.3048" layer="1"/>
+<wire x1="21" y1="8.7162" x2="21.8032" y2="9.5194" width="0.3048" layer="1"/>
 </signal>
 <signal name="N$2">
